File: KiCAD-Files/PD_trigger-board.kicad_pcb (KiCad board)
At the start: 2 copper layers, 18 x 23.5 mm, 16 parts, among them J1 USB_C_Receptacle_USB3.0_12P, U1 HUSB238, U2 SI4459ADY-T1-GE3, U3 ESP32-S3-mini_pinprofile

Commit message: smaller changes
Other:
- board text added: "PD-Trigger-Board PD 3.0"
- board text added: "v0.2"
- board text removed: "PD-Trigger-Board v0.2 PD V2.0"
Changed lines of the file:
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@@
 			(effects
 				(font
-					(size 0.75 0.75)
+					(size 0.5 0.5)
 					(thickness 0.1)
 				)
@@
 		(tags "USB 2.0 C Type-C Receptacle SMD 16P 16C USB4110-GF-A")
 		(property "Reference" "J1"
-			(at 0 -0.078 180)
+			(at 0 -0.078 0)
 			(unlocked yes)
 			(layer "F.SilkS")
 			(effects
 				(font
-					(size 0.75 0.75)
+					(size 0.5 0.5)
 					(thickness 0.1)
 				)
@@
 			(effects
 				(font
-					(size 0.75 0.75)
+					(size 0.5 0.5)
 					(thickness 0.1)
 				)
@@
 			(effects
 				(font
-					(size 0.75 0.75)
+					(size 0.5 0.5)
 					(thickness 0.1)
 				)
@@
 			(effects
 				(font
-					(size 0.75 0.75)
+					(size 0.5 0.5)
 					(thickness 0.1)
 				)
@@
 			(effects
 				(font
-					(size 0.75 0.75)
+					(size 0.5 0.5)
 					(thickness 0.1)
 				)
@@
 			(effects
 				(font
-					(size 0.75 0.75)
+					(size 0.5 0.5)
 					(thickness 0.1)
 				)
@@
 			(layer "F.Fab")
 		)
-		(fp_text user "${REFERENCE}"
-			(at 0 0 0)
-			(unlocked yes)
-			(layer "F.Fab")
+		(fp_text user "*"
+			(at -2.3176 -2.9316 0)
+			(layer "F.SilkS")
 			(effects
 				(font
@@
 			)
 		)
-		(fp_text user "*"
-			(at -1.6129 -2.4257 0)
+		(fp_text user "${REFERENCE}"
+			(at 0 0 0)
+			(unlocked yes)
 			(layer "F.Fab")
 			(effects
@@
 			(at -3.181 0.003 0)
 			(unlocked yes)
-			(layer "F.SilkS")
+			(layer "F.Fab")
 			(effects
 				(font
-					(size 1 1)
+					(size 0.5 0.5)
 					(thickness 0.1)
 				)
@@
 		(tags "capacitor")
 		(property "Reference" "C2"
-			(at 2.8 0 90)
-			(layer "F.SilkS")
+			(at 2.8316 0 90)
+			(layer "F.Fab")
 			(effects
 				(font
-					(size 0.75 0.75)
+					(size 0.5 0.5)
 					(thickness 0.1)
 				)
@@
 			(effects
 				(font
-					(size 0.75 0.75)
+					(size 0.5 0.5)
 					(thickness 0.1)
 				)
@@
 			(effects
 				(font
-					(size 0.75 0.75)
+					(size 0.5 0.5)
 					(thickness 0.1)
 				)
@@
 			(effects
 				(font
-					(size 0.75 0.75)
+					(size 0.5 0.5)
 					(thickness 0.1)
 				)
@@
 		(property "Reference" "C4"
 			(at 2.7 0 90)
-			(layer "F.SilkS")
+			(layer "F.Fab")
 			(effects
 				(font
-					(size 0.75 0.75)
+					(size 0.5 0.5)
 					(thickness 0.1)
 				)
@@
 		(property "Reference" "C3"
 			(at 2.8 0 90)
-			(layer "F.SilkS")
+			(layer "F.Fab")
 			(effects
 				(font
-					(size 0.75 0.75)
+					(size 0.5 0.5)
 					(thickness 0.1)
 				)
@@
 			(effects
 				(font
-					(size 0.75 0.75)
+					(size 0.5 0.5)
 					(thickness 0.1)
 				)
@@
 			(effects
 				(font
-					(size 0.75 0.75)
+					(size 0.5 0.5)
 					(thickness 0.1)
 				)
@@
 		(layer "F.SilkS")
 	)
-	(gr_text "PD-Trigger-Board v0.2\nPD V2.0"
-		(at 146.8 91.8 0)
+	(gr_text "PD-Trigger-Board\nPD 3.0"
+		(at 146.038 91.6984 0)
 		(layer "B.SilkS")
 		(effects
@@
 		)
 	)
+	(gr_text "v0.2"
+		(at 135.8646 89.281 0)
+		(layer "B.SilkS")
+		(effects
+			(font
+				(size 0.5 0.5)
+				(thickness 0.1)
+				(bold yes)
+			)
+			(justify left bottom mirror)
+		)
+	)
 	(gr_text "blinkyparts GmbH\nEgerstr. 9, RGB\nCC-BY-SA 4.0"
 		(at 144.9 80.7 0)
@@
 	)
 	(gr_text "20V"
-		(at 133.1 95.7 -90)
+		(at 133.3246 96.012 270)
 		(layer "F.SilkS")
 		(effects
 			(font
-				(size 0.75 0.75)
+				(size 0.5 0.5)
 				(thickness 0.1)
 			)
@@
 	)
 	(gr_text "9V"
-		(at 132.6 80.7 -90)
+		(at 132.9182 80.9498 270)
 		(layer "F.SilkS")
 		(effects
 			(font
-				(size 0.75 0.75)
+				(size 0.5 0.5)
 				(thickness 0.1)
 			)
@@
 	)
 	(gr_text "5V"
-		(at 132.6 78.2 -90)
+		(at 132.9182 78.4352 270)
 		(layer "F.SilkS")
 		(effects
 			(font
-				(size 0.75 0.75)
+				(size 0.5 0.5)
 				(thickness 0.1)
 			)
@@
 	)
 	(gr_text "15V"
-		(at 133.1 88.1 -90)
+		(at 133.2484 88.3666 270)
 		(layer "F.SilkS")
 		(effects
 			(font
-				(size 0.75 0.75)
+				(size 0.5 0.5)
 				(thickness 0.1)
 			)
@@
 	)
 	(gr_text "12V"
-		(at 133.1 85.5 -90)
+		(at 133.2484 85.8012 270)
 		(layer "F.SilkS")
 		(effects
 			(font
-				(size 0.75 0.75)
+				(size 0.5 0.5)
 				(thickness 0.1)
 			)
@@
 	)
 	(gr_text "18V"
-		(at 133.1 93.2 -90)
+		(at 133.2992 93.4974 270)
 		(layer "F.SilkS")
 		(effects
 			(font
-				(size 0.75 0.75)
+				(size 0.5 0.5)
 				(thickness 0.1)
 			)

Commit message: Minor design changes
Parts:
- moved C4 4.85 mm to (145.9, 92.9), turned to 90 degrees
- moved C3 2.95 mm to (145.9, 96.2)
- moved C2 2.55 mm to (144.2, 97.1)
- moved R3 0.06 mm to (136.4, 94.1)
Routing:
- net VBUS: track 6.80 -> 15.9 mm, vias 9 -> 5
- net GND: track 30.9 -> 22.7 mm, vias 18 -> 13
- net VOUT: track 19.0 -> 15.5 mm

Commit message: minor changes for v0.2
Parts:
- added ce-symbol_mask_3mm: G***, blinkyparts:ce-icon_3mm, B.Cu at (145.2, 90.2)
- added rohs-symbol_mask_3mm: G***, blinkyparts:rohs-icon_3mm, B.Cu at (139.0, 86.4)
- added weee-symbol_mask_3mm: G***, blinkyparts:weee-icon_3mm, B.Cu at (139.5, 90.8)
